Commit message: Added a new joint
all modification for the new joint.
the joint between original joint 2 and 3.

File: pro7a_description/urdf/pro7a_gazebo.urdf (robot description, URDF)
Before this commit: robot pro7a, 8 links, 7 joints
Links:
- added link end_link, mass 0.0062712; collision mesh filename=package://pro7a_description/meshes/end_link.STL; visual mesh filename=package://pro7a_description/meshes/end_link.STL
- link link1: geometry collision mesh filename=package://pro7a_description/meshes/link1.STL; visual mesh filename=package://pro7a_description/meshes/link1.STL
- link link2: mass 0.353299691884094 -> 0.35395; geometry collision mesh filename=package://pro7a_description/meshes/link2.STL; visual mesh filename=package://pro7a_description/meshes/link2.STL
- link link3: mass 0.500115096713792 -> 0.50149; geometry collision mesh filename=package://pro7a_description/meshes/link3.STL; visual mesh filename=package://pro7a_description/meshes/link3.STL
- link link4: mass 0.494453076498356 -> 0.53361; geometry collision mesh filename=package://pro7a_description/meshes/link4.STL; visual mesh filename=package://pro7a_description/meshes/link4.STL
- link link5: mass 0.355062206783252 -> 0.35861; geometry collision mesh filename=package://pro7a_description/meshes/link5.STL; visual mesh filename=package://pro7a_description/meshes/link5.STL
- link link6: mass 0.200934163479789 -> 0.2022; geometry collision mesh filename=package://pro7a_description/meshes/link6.STL; visual mesh filename=package://pro7a_description/meshes/link6.STL
- link link7: mass 0.162169114093039 -> 0.16217; geometry collision mesh filename=package://pro7a_description/meshes/link7.STL; visual mesh filename=package://pro7a_description/meshes/link7.STL
Joints:
- added joint joint7: type revolute, parent link7, child end_link, origin xyz=0 0.048 0.123 rpy=0 0 0, axis 0 0 1, limit lower=-2.62 upper=2.62 effort=1000 velocity=6.5
- joint joint1: limit lower=-2.094395102 upper=2.094395102 effort=1000 velocity=6.5 -> lower=-2.62 upper=2.62 effort=1000 velocity=6.5
- joint joint2: origin xyz=0 -0.072 0.033 rpy=0 0 0 -> xyz=0 -0.072 0.034 rpy=0 0 0
- joint joint3: limit lower=-2.094395102 upper=2.094395102 effort=1000 velocity=6.5 -> lower=-2.62 upper=2.62 effort=1000 velocity=6.5; origin xyz=0 0.072 0.1933 rpy=0 0 0 -> xyz=0 0.072 0.195 rpy=0 0 0
- joint joint4: axis 0 -1 0 -> 0 1 0; limit lower=-3.141592654 upper=0.65 effort=1000 velocity=6.5 -> lower=-0.65 upper=3.141592654 effort=1000 velocity=6.5; origin xyz=0.03 -0.060 0.093 rpy=0.0 0.0 0.0 -> xyz=0.03 -0.06 0.095 rpy=0 0 0
- joint joint5: limit lower=-2.094395102 upper=2.094395102 effort=1000 velocity=6.5 -> lower=-2.62 upper=2.62 effort=1000 velocity=6.5
- joint joint6: axis 0 -1 0 -> 0 1 0
